File: Hardware/Qwiic-USB_Hub.sch (EAGLE design)
At the start: 61 parts, among them J1 USB_A_FEMALE, J2 Qwiic Right Angle, J3 PTH, J4 Qwiic Right Angle, J6 USB_A_FEMALE, J8 USB_A_FEMALE, J9 USB_A_FEMALE, Q1 4.3A/20V/54mΩ, Q2 4.3A/20V/54mΩ, Q3 4.3A/20V/54mΩ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

Commit message: Fixing silk typo in OCS labels. Adding production panels.
Parts:
- added D1: 3A/10V/280mV, SparkFun-DiscreteSemi:DIODE-SCHOTTKY-BAT60A
Connections:
- net D+ renamed D_P
- net D- renamed D_N
- net PORT1_DM renamed PORT1_N
- net PORT1_DP renamed PORT1_P
- net PORT2_DM renamed PORT2_N
- net PORT2_DP renamed PORT2_P
- net PORT3_DM renamed PORT3_N
- net PORT3_DP renamed PORT3_P
- net PORT4_DM renamed PORT4_N
- net PORT4_DP renamed PORT4_P
- new net N$21: D1.A, J2.2, J3.VCC, J4.2
- net 3.3V: now also D1.C; no longer J2.2, J3.VCC, J4.2
Changed lines of the file:
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@@
 <part name="JP21" library="SparkFun" deviceset="FIDUCIAL" device="UFIDUCIAL"/>
 <part name="JP61" library="SparkFun" deviceset="FIDUCIAL" device="UFIDUCIAL"/>
-<part name="SUPPLY4" library="SparkFun-PowerSymbols" deviceset="3.3V" device=""/>
 <part name="J2" library="SparkFun-Connectors" deviceset="I2C_STANDARD" device="QWIIC" value="Qwiic Right Angle"/>
-<part name="SUPPLY7" library="SparkFun-PowerSymbols" deviceset="3.3V" device=""/>
 <part name="J3" library="SparkX" deviceset="I2C_STANDARD" device="_NO_SILK" value="PTH"/>
-<part name="SUPPLY8" library="SparkFun-PowerSymbols" deviceset="3.3V" device=""/>
 <part name="J4" library="SparkFun-Connectors" deviceset="I2C_STANDARD" device="QWIIC" value="Qwiic Right Angle"/>
 <part name="LOGO1" library="SparkFun-Aesthetics" deviceset="OSHW-LOGO" device="MINI"/>
@@
 <part name="R14" library="SparkFun-Resistors" deviceset="22OHM" device="-0603-1/10W-1%" value="22"/>
 <part name="R15" library="SparkFun-Resistors" deviceset="22OHM" device="-0603-1/10W-1%" value="22"/>
+<part name="D1" library="SparkFun-DiscreteSemi" deviceset="DIODE-SCHOTTKY" device="-BAT60A" value="3A/10V/280mV"/>
+<part name="SUPPLY4" library="SparkFun-PowerSymbols" deviceset="3.3V" device=""/>
 </parts>
 <sheets>
@@
 <instance part="JP21" gate="G$1" x="416.56" y="33.02" smashed="yes" rot="R270"/>
 <instance part="JP61" gate="G$1" x="419.1" y="33.02" smashed="yes"/>
-<instance part="SUPPLY4" gate="G$1" x="25.4" y="83.82" smashed="yes">
-<attribute name="VALUE" x="25.4" y="86.614" size="1.778" layer="96" align="bottom-center"/>
-</instance>
 <instance part="J2" gate="G$1" x="35.56" y="76.2" smashed="yes" rot="MR0">
 <attribute name="VALUE" x="43.434" y="91.44" size="1.778" layer="96" font="vector" rot="MR270" align="top-left"/>
 <attribute name="NAME" x="40.64" y="84.074" size="1.778" layer="95" font="vector" rot="MR0"/>
 </instance>
-<instance part="SUPPLY7" gate="G$1" x="25.4" y="30.48" smashed="yes">
-<attribute name="VALUE" x="25.4" y="33.274" size="1.778" layer="96" align="bottom-center"/>
-</instance>
 <instance part="J3" gate="G$1" x="35.56" y="22.86" smashed="yes" rot="MR0">
 <attribute name="VALUE" x="40.64" y="17.526" size="1.778" layer="96" font="vector" rot="MR0" align="top-left"/>
 <attribute name="NAME" x="40.64" y="30.734" size="1.778" layer="95" font="vector" rot="MR0"/>
-</instance>
-<instance part="SUPPLY8" gate="G$1" x="25.4" y="55.88" smashed="yes">
-<attribute name="VALUE" x="25.4" y="58.674" size="1.778" layer="96" align="bottom-center"/>
 </instance>
 <instance part="J4" gate="G$1" x="35.56" y="48.26" smashed="yes" rot="MR0">
@@
 <attribute name="VALUE" x="129.54" y="134.366" size="1.778" layer="96" align="top-center"/>
 </instance>
-<instance part="GND6" gate="1" x="25.4" y="68.58" smashed="yes" rot="MR0">
-<attribute name="VALUE" x="25.4" y="68.326" size="1.778" layer="96" rot="MR0" align="top-center"/>
-</instance>
-<instance part="GND7" gate="1" x="25.4" y="40.64" smashed="yes" rot="MR0">
-<attribute name="VALUE" x="25.4" y="40.386" size="1.778" layer="96" rot="MR0" align="top-center"/>
+<instance part="GND6" gate="1" x="22.86" y="68.58" smashed="yes" rot="MR0">
+<attribute name="VALUE" x="22.86" y="68.326" size="1.778" layer="96" rot="MR0" align="top-center"/>
+</instance>
+<instance part="GND7" gate="1" x="22.86" y="40.64" smashed="yes" rot="MR0">
+<attribute name="VALUE" x="22.86" y="40.386" size="1.778" layer="96" rot="MR0" align="top-center"/>
 </instance>
 <instance part="GND8" gate="1" x="25.4" y="15.24" smashed="yes" rot="MR0">
@@
 <attribute name="NAME" x="99.568" y="226.06" size="1.778" layer="95" font="vector" align="bottom-center"/>
 <attribute name="VALUE" x="108.458" y="226.314" size="1.778" layer="96" font="vector" rot="R180" align="top-center"/>
+</instance>
+<instance part="D1" gate="G$1" x="25.4" y="86.36" smashed="yes" rot="R90">
+<attribute name="NAME" x="20.066" y="88.138" size="1.778" layer="95" font="vector"/>
+<attribute name="VALUE" x="3.81" y="87.122" size="1.778" layer="96" font="vector" align="top-left"/>
+</instance>
+<instance part="SUPPLY4" gate="G$1" x="25.4" y="91.44" smashed="yes">
+<attribute name="VALUE" x="25.4" y="94.234" size="1.778" layer="96" align="bottom-center"/>
 </instance>
 </instances>
@@
 <nets>
 <net name="3.3V" class="2">
-<segment>
-<pinref part="J2" gate="G$1" pin="2"/>
-<wire x1="27.94" y1="76.2" x2="25.4" y2="76.2" width="0.1524" layer="91"/>
-<wire x1="25.4" y1="76.2" x2="25.4" y2="83.82" width="0.1524" layer="91"/>
-<pinref part="SUPPLY4" gate="G$1" pin="3.3V"/>
-</segment>
-<segment>
-<pinref part="J3" gate="G$1" pin="VCC"/>
-<wire x1="27.94" y1="22.86" x2="25.4" y2="22.86" width="0.1524" layer="91"/>
-<wire x1="25.4" y1="22.86" x2="25.4" y2="30.48" width="0.1524" layer="91"/>
-<pinref part="SUPPLY7" gate="G$1" pin="3.3V"/>
-</segment>
-<segment>
-<pinref part="J4" gate="G$1" pin="2"/>
-<wire x1="27.94" y1="48.26" x2="25.4" y2="48.26" width="0.1524" layer="91"/>
-<wire x1="25.4" y1="48.26" x2="25.4" y2="55.88" width="0.1524" layer="91"/>
-<pinref part="SUPPLY8" gate="G$1" pin="3.3V"/>
-</segment>
 <segment>
 <wire x1="114.3" y1="149.86" x2="119.38" y2="149.86" width="0.1524" layer="91"/>
@@
 <pinref part="SUPPLY15" gate="G$1" pin="3.3V"/>
 </segment>
+<segment>
+<pinref part="D1" gate="G$1" pin="C"/>
+<wire x1="25.4" y1="88.9" x2="25.4" y2="91.44" width="0.1524" layer="91"/>
+<pinref part="SUPPLY4" gate="G$1" pin="3.3V"/>
+</segment>
 </net>
 <net name="GND" class="0">
@@
 <segment>
 <pinref part="J2" gate="G$1" pin="1"/>
-<wire x1="27.94" y1="73.66" x2="25.4" y2="73.66" width="0.1524" layer="91"/>
-<wire x1="25.4" y1="73.66" x2="25.4" y2="71.12" width="0.1524" layer="91"/>
+<wire x1="27.94" y1="73.66" x2="22.86" y2="73.66" width="0.1524" layer="91"/>
+<wire x1="22.86" y1="73.66" x2="22.86" y2="71.12" width="0.1524" layer="91"/>
 <pinref part="GND6" gate="1" pin="GND"/>
 </segment>
 <segment>
 <pinref part="J4" gate="G$1" pin="1"/>
-<wire x1="27.94" y1="45.72" x2="25.4" y2="45.72" width="0.1524" layer="91"/>
-<wire x1="25.4" y1="45.72" x2="25.4" y2="43.18" width="0.1524" layer="91"/>
+<wire x1="27.94" y1="45.72" x2="22.86" y2="45.72" width="0.1524" layer="91"/>
+<wire x1="22.86" y1="45.72" x2="22.86" y2="43.18" width="0.1524" layer="91"/>
 <pinref part="GND7" gate="1" pin="GND"/>
 </segment>
@@
 </segment>
 </net>
-<net name="D+" class="0">
+<net name="D_P" class="0">
 <segment>
 <wire x1="68.58" y1="144.78" x2="73.66" y2="144.78" width="0.1524" layer="91"/>
@@
 </segment>
 </net>
-<net name="D-" class="0">
+<net name="D_N" class="0">
 <segment>
 <wire x1="68.58" y1="134.62" x2="73.66" y2="134.62" width="0.1524" layer="91"/>
@@
 </segment>
 </net>
-<net name="PORT1_DM" class="0">
+<net name="PORT1_N" class="0">
 <segment>
 <pinref part="U1" gate="U1" pin="USBDM_DN1"/>
@@
 </segment>
 </net>
-<net name="PORT1_DP" class="0">
+<net name="PORT1_P" class="0">
 <segment>
 <pinref part="U1" gate="U1" pin="USBDP_DN1"/>
@@
 </segment>
 </net>
-<net name="PORT2_DM" class="0">
+<net name="PORT2_N" class="0">
 <segment>
 <pinref part="U1" gate="U1" pin="USBDM_DN2"/>
@@
 </segment>
 </net>
-<net name="PORT2_DP" class="0">
+<net name="PORT2_P" class="0">
 <segment>
 <pinref part="U1" gate="U1" pin="USBDP_DN2"/>
@@
 </segment>
 </net>
-<net name="PORT3_DM" class="0">
+<net name="PORT3_N" class="0">
 <segment>
 <pinref part="U1" gate="U1" pin="USBDM_DN3"/>
@@
 </segment>
 </net>
-<net name="PORT3_DP" class="0">
+<net name="PORT3_P" class="0">
 <segment>
 <pinref part="U1" gate="U1" pin="USBDP_DN3"/>
@@
 </segment>
 </net>
-<net name="PORT4_DM" class="0">
+<net name="PORT4_N" class="0">
 <segment>
 <pinref part="U1" gate="U1" pin="USBDM_DN4"/>
@@
 </segment>
 </net>
-<net name="PORT4_DP" class="0">
+<net name="PORT4_P" class="0">
 <segment>
 <pinref part="U1" gate="U1" pin="USBDP_DN4"/>
@@
 </segment>
 </net>
+<net name="N$21" class="2">
+<segment>
+<pinref part="J3" gate="G$1" pin="VCC"/>
+<wire x1="27.94" y1="22.86" x2="25.4" y2="22.86" width="0.1524" layer="91"/>
+<pinref part="J4" gate="G$1" pin="2"/>
+<wire x1="27.94" y1="48.26" x2="25.4" y2="48.26" width="0.1524" layer="91"/>
+<wire x1="25.4" y1="22.86" x2="25.4" y2="48.26" width="0.1524" layer="91"/>
+<junction x="25.4" y="48.26"/>
+<pinref part="J2" gate="G$1" pin="2"/>
+<wire x1="27.94" y1="76.2" x2="25.4" y2="76.2" width="0.1524" layer="91"/>
+<wire x1="25.4" y1="76.2" x2="25.4" y2="83.82" width="0.1524" layer="91"/>
+<wire x1="25.4" y1="48.26" x2="25.4" y2="76.2" width="0.1524" layer="91"/>
+<junction x="25.4" y="76.2"/>
+<pinref part="D1" gate="G$1" pin="A"/>
+</segment>
+</net>

Commit message: Add connections to config pins.
Parts:
- J10: device SparkFun-Connectors:CONN_08NO_SILK_FEMALE_PTH -> SparkFun-Connectors:CONN_10NO_SILK_PTH_FEMALE
- JP5: value JUMPER-SMT_3_2-NC_TRACE_SILK -> JUMPER-SMT_3_NO_SILK; device SparkFun-Jumpers:JUMPER-SMT_3_2-NC_TRACE_SILK -> SparkFun-Jumpers:JUMPER-SMT_3_NO_SILK
Connections:
- removed net N$12: R4.2, U1.HS_IND
- removed net SCL: J2.4, J3.SCL, J4.4, R13.1, U1.SCL
- new net CFG1: J10.7, R4.2, U1.HS_IND/CFG1
- new net SCL/CFG0: J10.8, J2.4, J3.SCL, J4.4, R13.1, U1.SCL/CFG0
- net 3.3V: now also J10.9; no longer J10.7
- net 5V: now also J10.10; no longer J10.8
Other:
- note added: "J5: Open (Default) - Boot as Hub / Default Config Closed - Require I2C Configuration"
Changed lines of the file:
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@@
 <part name="R12" library="SparkFun-Resistors" deviceset="2.2KOHM" device="-0603-1/10W-1%" value="2.2k"/>
 <part name="R13" library="SparkFun-Resistors" deviceset="2.2KOHM" device="-0603-1/10W-1%" value="2.2k"/>
-<part name="JP5" library="SparkFun-Jumpers" deviceset="JUMPER-SMT_3_2-NC_TRACE" device="_SILK" package3d_urn="urn:adsk.eagle:package:39289/1" value=""/>
+<part name="JP5" library="SparkFun-Jumpers" deviceset="JUMPER-SMT_3_NO" device="_SILK" package3d_urn="urn:adsk.eagle:package:39285/1" value=""/>
 <part name="SUPPLY15" library="SparkFun-PowerSymbols" deviceset="3.3V" device=""/>
 <part name="LOGO2" library="SparkFun-Aesthetics" deviceset="QWIIC_LOGO" device="_CONNECTOR"/>
-<part name="J10" library="SparkFun-Connectors" deviceset="CONN_08" device="NO_SILK_FEMALE_PTH"/>
 <part name="U$5" library="SparkX" deviceset="SPARKX-LOGO" device="4"/>
 <part name="SUPPLY16" library="SparkFun-PowerSymbols" deviceset="5V" device=""/>
@@
 <part name="D1" library="SparkFun-DiscreteSemi" deviceset="DIODE-SCHOTTKY" device="-BAT60A" value="3A/10V/280mV"/>
 <part name="SUPPLY4" library="SparkFun-PowerSymbols" deviceset="3.3V" device=""/>
+<part name="J10" library="SparkFun-Connectors" deviceset="CONN_10" device="NO_SILK_PTH_FEMALE"/>
 </parts>
 <sheets>
@@
 <wire x1="0" y1="180.34" x2="185.42" y2="180.34" width="0.2032" layer="97" style="longdash"/>
 <wire x1="185.42" y1="180.34" x2="185.42" y2="279.4" width="0.2032" layer="97" style="longdash"/>
-<wire x1="124.46" y1="101.6" x2="0" y2="101.6" width="0.2032" layer="97" style="longdash"/>
+<wire x1="185.42" y1="101.6" x2="0" y2="101.6" width="0.2032" layer="97" style="longdash"/>
 <wire x1="185.42" y1="180.34" x2="185.42" y2="101.6" width="0.2032" layer="97" style="longdash"/>
-<wire x1="185.42" y1="101.6" x2="124.46" y2="101.6" width="0.2032" layer="97" style="longdash"/>
-<wire x1="124.46" y1="101.6" x2="124.46" y2="0" width="0.2032" layer="97" style="longdash"/>
+<wire x1="185.42" y1="101.6" x2="185.42" y2="0" width="0.2032" layer="97" style="longdash"/>
 <text x="93.98" y="269.24" size="2.54" layer="94" rot="MR180" align="center">USB Hub</text>
 <text x="73.66" y="162.56" size="2.54" layer="94" rot="MR180" align="center">USB / Power</text>
@@
 <text x="30.48" y="167.64" size="1.778" layer="97" font="vector" align="center">Closing jumper bypasses PTC
 to allow &gt;2A current flows.</text>
+<text x="111.76" y="86.36" size="1.778" layer="97" align="center-left">J5:
+Open (Default) - Boot as Hub / Default Config
+Closed - Require I2C Configuration</text>
 </plain>
 <instances>
@@
 <instance part="JP91" gate="G$1" x="426.72" y="33.02" smashed="yes"/>
 <instance part="JP101" gate="G$1" x="426.72" y="30.48" smashed="yes"/>
-<instance part="GND1" gate="1" x="66.04" y="35.56" smashed="yes" rot="MR0">
-<attribute name="VALUE" x="66.04" y="35.306" size="1.778" layer="96" rot="MR0" align="top-center"/>
+<instance part="GND1" gate="1" x="66.04" y="30.48" smashed="yes" rot="MR0">
+<attribute name="VALUE" x="66.04" y="30.226" size="1.778" layer="96" rot="MR0" align="top-center"/>
 </instance>
 <instance part="C4" gate="G$1" x="119.38" y="142.24" smashed="yes">
@@
 </instance>
 <instance part="LOGO2" gate="G$1" x="393.7" y="40.64" smashed="yes"/>
-<instance part="J10" gate="G$1" x="73.66" y="48.26" smashed="yes" rot="MR0">
-<attribute name="VALUE" x="78.74" y="35.814" size="1.778" layer="96" font="vector" rot="MR0"/>
-<attribute name="NAME" x="78.74" y="61.468" size="1.778" layer="95" font="vector" rot="MR0"/>
-</instance>
 <instance part="U$5" gate="G$1" x="393.7" y="48.26" smashed="yes"/>
 <instance part="SUPPLY16" gate="G$1" x="10.16" y="254" smashed="yes">
@@
 <instance part="SUPPLY4" gate="G$1" x="25.4" y="91.44" smashed="yes">
 <attribute name="VALUE" x="25.4" y="94.234" size="1.778" layer="96" align="bottom-center"/>
+</instance>
+<instance part="J10" gate="J1" x="78.74" y="53.34" smashed="yes" rot="MR0">
+<attribute name="VALUE" x="78.74" y="30.734" size="1.778" layer="96" font="vector" rot="MR0"/>
+<attribute name="NAME" x="78.74" y="61.468" size="1.778" layer="95" font="vector" rot="MR0"/>
 </instance>
 </instances>
@@
 <pinref part="SUPPLY10" gate="G$1" pin="3.3V"/>
 <wire x1="60.96" y1="55.88" x2="60.96" y2="60.96" width="0.1524" layer="91"/>
-<pinref part="J10" gate="G$1" pin="7"/>
+<pinref part="J10" gate="J1" pin="9"/>
 </segment>
 <segment>
@@
 <segment>
 <pinref part="GND1" gate="1" pin="GND"/>
-<wire x1="68.58" y1="40.64" x2="66.04" y2="40.64" width="0.1524" layer="91"/>
-<wire x1="66.04" y1="40.64" x2="66.04" y2="38.1" width="0.1524" layer="91"/>
-<pinref part="J10" gate="G$1" pin="1"/>
+<wire x1="68.58" y1="35.56" x2="66.04" y2="35.56" width="0.1524" layer="91"/>
+<wire x1="66.04" y1="35.56" x2="66.04" y2="33.02" width="0.1524" layer="91"/>
+<pinref part="J10" gate="J1" pin="1"/>
 </segment>
 <segment>
@@
 </segment>
 <segment>
-<wire x1="68.58" y1="53.34" x2="66.04" y2="53.34" width="0.1524" layer="91"/>
-<label x="66.04" y="53.34" size="1.27" layer="95" rot="R180" xref="yes"/>
-<pinref part="J10" gate="G$1" pin="6"/>
+<wire x1="68.58" y1="48.26" x2="66.04" y2="48.26" width="0.1524" layer="91"/>
+<label x="66.04" y="48.26" size="1.27" layer="95" rot="R180" xref="yes"/>
+<pinref part="J10" gate="J1" pin="6"/>
 </segment>
 </net>
@@
 <pinref part="SUPPLY11" gate="G$1" pin="5V"/>
 <wire x1="66.04" y1="58.42" x2="66.04" y2="60.96" width="0.1524" layer="91"/>
-<pinref part="J10" gate="G$1" pin="8"/>
+<pinref part="J10" gate="J1" pin="10"/>
 </segment>
 <segment>
@@
 </segment>
 </net>
-<net name="SCL" class="0">
-<segment>
-<pinref part="U1" gate="U1" pin="SCL"/>
+<net name="SCL/CFG0" class="0">
+<segment>
+<pinref part="U1" gate="U1" pin="SCL/CFG0"/>
 <wire x1="111.76" y1="223.52" x2="109.22" y2="223.52" width="0.1524" layer="91"/>
 <label x="109.22" y="223.52" size="1.27" layer="95" rot="R180" xref="yes"/>
@@
 <wire x1="114.3" y1="66.04" x2="111.76" y2="66.04" width="0.1524" layer="91"/>
 <label x="111.76" y="66.04" size="1.27" layer="95" rot="R180" xref="yes"/>
+</segment>
+<segment>
+<wire x1="68.58" y1="53.34" x2="66.04" y2="53.34" width="0.1524" layer="91"/>
+<label x="66.04" y="53.34" size="1.27" layer="95" rot="R180" xref="yes"/>
+<pinref part="J10" gate="J1" pin="8"/>
 </segment>
 </net>
@@
 </segment>
 </net>
-<net name="N$12" class="0">
-<segment>
-<pinref part="U1" gate="U1" pin="HS_IND"/>
+<net name="CFG1" class="0">
+<segment>
+<pinref part="U1" gate="U1" pin="HS_IND/CFG1"/>
 <pinref part="R4" gate="G$1" pin="2"/>
 <wire x1="111.76" y1="243.84" x2="68.58" y2="243.84" width="0.1524" layer="91"/>
 <wire x1="68.58" y1="243.84" x2="68.58" y2="236.22" width="0.1524" layer="91"/>
+<label x="66.04" y="243.84" size="1.27" layer="95" rot="R180" xref="yes"/>
+<wire x1="68.58" y1="243.84" x2="66.04" y2="243.84" width="0.1524" layer="91"/>
+<junction x="68.58" y="243.84"/>
+</segment>
+<segment>
+<wire x1="68.58" y1="50.8" x2="66.04" y2="50.8" width="0.1524" layer="91"/>
+<label x="66.04" y="50.8" size="1.27" layer="95" rot="R180" xref="yes"/>
+<pinref part="J10" gate="J1" pin="7"/>
 </segment>
 </net>
@@
 </segment>
 <segment>
-<wire x1="68.58" y1="50.8" x2="66.04" y2="50.8" width="0.1524" layer="91"/>
-<label x="66.04" y="50.8" size="1.27" layer="95" rot="R180" xref="yes"/>
-<pinref part="J10" gate="G$1" pin="5"/>
+<wire x1="68.58" y1="45.72" x2="66.04" y2="45.72" width="0.1524" layer="91"/>
+<label x="66.04" y="45.72" size="1.27" layer="95" rot="R180" xref="yes"/>
+<pinref part="J10" gate="J1" pin="5"/>
 </segment>
 </net>
@@
 </segment>
 <segment>
-<wire x1="68.58" y1="48.26" x2="66.04" y2="48.26" width="0.1524" layer="91"/>
-<label x="66.04" y="48.26" size="1.27" layer="95" rot="R180" xref="yes"/>
-<pinref part="J10" gate="G$1" pin="4"/>
+<wire x1="68.58" y1="43.18" x2="66.04" y2="43.18" width="0.1524" layer="91"/>
+<label x="66.04" y="43.18" size="1.27" layer="95" rot="R180" xref="yes"/>
+<pinref part="J10" gate="J1" pin="4"/>
 </segment>
 </net>
@@
 </segment>
 <segment>
-<wire x1="68.58" y1="45.72" x2="66.04" y2="45.72" width="0.1524" layer="91"/>
-<label x="66.04" y="45.72" size="1.27" layer="95" rot="R180" xref="yes"/>
-<pinref part="J10" gate="G$1" pin="3"/>
+<wire x1="68.58" y1="40.64" x2="66.04" y2="40.64" width="0.1524" layer="91"/>
+<label x="66.04" y="40.64" size="1.27" layer="95" rot="R180" xref="yes"/>
+<pinref part="J10" gate="J1" pin="3"/>
 </segment>
 </net>
@@
 </segment>
 <segment>
-<wire x1="68.58" y1="43.18" x2="66.04" y2="43.18" width="0.1524" layer="91"/>
-<label x="66.04" y="43.18" size="1.27" layer="95" rot="R180" xref="yes"/>
-<pinref part="J10" gate="G$1" pin="2"/>
-</segment>
-</net>
+<wire x1="68.58" y1="38.1" x2="66.04" y2="38.1" width="0.1524" layer="91"/>
+<label x="66.04" y="38.1" size="1.27" layer="95" rot="R180" xref="yes"/>
+<pinref part="J10" gate="J1" pin="2"/>
+</segment>
+</net>
