File: Hardware/Production/Qwiic-USB_Hub-Panel.brd (EAGLE design)
At the start: 189.2 x 95 mm, 321 parts, among them J1 USB_A_FEMALE, J11 PTH, J12 Qwiic Right Angle, J14 USB_A_FEMALE, J15 USB_A_FEMALE, J16 USB_A_FEMALE, J17 USB_A_FEMALE, J19 Qwiic Right Angle, J2 Qwiic Right Angle, J20 PTH, J21 Qwiic Right Angle, J23 USB_A_FEMALE, J24 USB_A_FEMALE, J25 USB_A_FEMALE, J26 USB_A_FEMALE, J3 PTH, J4 Qwiic Right Angle, J6 USB_A_FEMALE, J7 Qwiic Right Angle, J8 USB_A_FEMALE, J9 USB_A_FEMALE, Q1 4.3A/20V/54mΩ, Q10 4.3A/20V/54mΩ, Q11 4.3A/20V/54mΩ, Q12 4.3A/20V/54mΩ, Q2 4.3A/20V/54mΩ, Q3 4.3A/20V/54mΩ, Q4 4.3A/20V/54mΩ, Q5 4.3A/20V/54mΩ, Q6 4.3A/20V/54mΩ, Q7 4.3A/20V/54mΩ, Q8 4.3A/20V/54mΩ, Q9 4.3A/20V/54mΩ, U1 USB251XB, U2 3.3V, U3 3.3V, U4 USB251XB, U5 3.3V, U6 USB251XB, Y1 24MHz, Y2 24MHz, Y3 24MHz

Commit message: Increase x02 panel size.
Parts:
- added BYP3, BYP4, BYP5: JUMPER-SMT_2_NO_SILK, SparkFun-Jumpers:SMT-JUMPER_2_NO_SILK
- added C28, C30, C37, C39, C46, C48: 1.0uF, SparkFun-Capacitors:0603
- added C29, C33, C34, C35, C36, C38, C42, C43, C44, C45, C47, C51, C52, C53, C54: 0.1uF, SparkFun-Capacitors:0603
- added C31, C32, C40, C41, C49, C50: 18pF, SparkFun-Capacitors:0603
- added D10, D12, D8: 3A/10V/280mV, SparkFun-DiscreteSemi:SOD-323
- added D11, D7, D9: PRTR5V0U2F, SparkFun-IC-Power:SOT886
- added F4, F5, F6: 6V/2A, SparkFun-Fuses:1210
- added J28, J30, J37, J39, J46, J48: Qwiic Right Angle, SparkFun-Connectors:JST04_1MM_RA
- added J29, J38, J47: PTH, SparkX:1X04_NO_SILK
- added J31, J40, J49: (no value), SparkFun-Connectors:USB-C-16P-2LAYER-PADS
- added J32, J33, J34, J35, J41, J42, J43, J44, J50, J51, J52, J53: USB_A_FEMALE, SparkFun-Connectors:USB-A-S-NOSILK-FEMALE
- added J36, J45, J54: (no value), SparkFun-Connectors:1X10_NO_SILK
- added JP20, JP22, JP27, JP28, JP30, JP32, JP37, JP38, JP40, JP42, JP47, JP48: STAND-OFF, SparkFun:STAND-OFF
- added JP23, JP24, JP25, JP26, JP33, JP34, JP35, JP36, JP43, JP44, JP45, JP46: FIDUCIALUFIDUCIAL, SparkFun:MICRO-FIDUCIAL
- added JP29, JP39, JP49: (no value), SparkFun-Jumpers:SMT-JUMPER_3_NO_SILK
- added LED4, LED5, LED6: RED, SparkFun-LED:LED-0603
- added LOGO10, LOGO12, LOGO8: QWIIC_LOGO_CONNECTOR, SparkFun-Aesthetics:QWIIC_5.5MM
- added LOGO11, LOGO7, LOGO9: OSHW-LOGOMINI, SparkFun-Aesthetics:OSHW-LOGO-MINI
- added PWR3, PWR4, PWR5: (no value), SparkFun-Jumpers:SMT-JUMPER_2_NC_TRACE_SILK
- added Q13, Q14, Q15, Q16, Q17, Q18, Q19, Q20, Q21, Q22, Q23, Q24: 4.3A/20V/54mΩ, SparkFun-DiscreteSemi:SOT23-3
- added R100, R101, R102, R103, R104, R60, R61, R62, R63, R64, R65, R66, R67, R68, R78, R79, R80, R81, R82, R83, R84, R85, R86, R96, R97, R98, R99: 100k, SparkFun-Resistors:0603
- added R105, R106, R69, R70, R87, R88: 2.2k, SparkFun-Resistors:0603
- added R107, R108, R71, R72, R89, R90: 22, SparkFun-Resistors:0603
- added R55, R73, R91: 1k, SparkFun-Resistors:0603
- added R56, R57, R74, R75, R92, R93: 5.1k, SparkFun-Resistors:0603
- added R58, R76, R94: 12k, SparkFun-Resistors:0603
- added R59, R77, R95: 1M, SparkFun-Resistors:0603
- added U$136, U$181, U$226: (no value), output:PORT40
- added U$137, U$182, U$227: (no value), output:PORT31
- added U$138, U$183, U$228: (no value), output:PORT22
- added U$139, U$184, U$229: (no value), output:PORT13
- added U$140, U$164, U$185, U$209, U$230, U$254: SPARKX-LOGO4, SparkX:SPARKX-MEDIUM
- added U$141, U$144, U$186, U$189, U$231, U$234: (no value), output:#3#3V#0
- added U$142, U$145, U$187, U$190, U$232, U$235: (no value), output:#SDA#0
- added U$143, U$146, U$188, U$191, U$233, U$236: (no value), output:#SCL#0
- added U$147, U$148, U$192, U$193, U$237, U$238: (no value), output:#GND#0
- added U$149, U$194, U$239: (no value), output:#I�C#1
- added U$150, U$195, U$240: (no value), output:PWR0
- added U$151, U$161, U$196, U$206, U$241, U$251: (no value), output:##RST##4
- added U$152, U$162, U$197, U$207, U$242, U$252: (no value), output:#3#3V#6
- added U$153, U$163, U$198, U$208, U$243, U$253: (no value), output:#5V#7
- added U$154, U$160, U$199, U$205, U$244, U$250: (no value), output:#GND#5
- added U$155, U$200, U$245: (no value), output:#BYP#0
- added U$156, U$167, U$201, U$212, U$246, U$257: (no value), output:USB2514B0
- added U$157, U$165, U$202, U$210, U$247, U$255: (no value), output:QWIIC2
- added U$158, U$166, U$203, U$211, U$248, U$256: (no value), output:USB_HUB1
- added U$159, U$204, U$249: (no value), output:#LED#0
- added U$168, U$213, U$258: (no value), SparkFun-Aesthetics:QWIIC_5.5MM
- added U$169, U$177, U$214, U$222, U$259, U$267: (no value), output:##OCS1##3
- added U$170, U$178, U$215, U$223, U$260, U$268: (no value), output:##OCS2##2
- added U$171, U$179, U$216, U$224, U$261, U$269: (no value), output:##OCS3##1
- added U$172, U$180, U$217, U$225, U$262, U$270: (no value), output:##OCS4##0
- added U$173, U$176, U$218, U$221, U$263, U$266: (no value), output:#CFG0#1
- added U$174, U$175, U$219, U$220, U$264, U$265: (no value), output:#CFG1#0
- added U10, U12, U8: USB251XB, USB251xB:QFN-36
- added U11, U7, U9: 3.3V, SparkFun-IC-Power:SOT23-5
- added Y4, Y5, Y6: 24MHz, SparkFun-Clocks:CRYSTAL-SMD-2.0X1.6MM
- moved E$1 81.8 mm to (-12.3, 160.4)
- moved E$2 81.8 mm to (-12.3, 160.4)
- moved E$3 81.8 mm to (162.1, 160.4)
- moved E$4 81.8 mm to (162.1, 160.4)
Connections:
- new net !OCS13: J36.5, U8.13
- new net !OCS14: J36.4, U8.17
- new net !OCS15: J36.3, U8.19
- new net !OCS16: J36.2, U8.21
- new net !OCS17: J45.5, U10.13
- new net !OCS18: J45.4, U10.17
- new net !OCS19: J45.3, U10.19
- new net !OCS20: J45.2, U10.21
- new net !OCS21: J54.5, U12.13
- new net !OCS22: J54.4, U12.17
- new net !OCS23: J54.3, U12.19
- new net !OCS24: J54.2, U12.21
- new net !RESET3: C35.1, J36.6, R62.1, U8.26
- new net !RESET4: C44.1, J45.6, R80.1, U10.26
- new net !RESET5: C53.1, J54.6, R98.1, U12.26
- new net 3.3V3: C28.1, C29.2, D8.C, J36.9, JP29.2, PWR3.2, R62.2, U7.5, U8.10, U8.15, U8.23, U8.29, U8.36, U8.5
- new net 3.3V4: C37.1, C38.2, D10.C, J45.9, JP39.2, PWR4.2, R80.2, U10.10, U10.15, U10.23, U10.29, U10.36, U10.5, U9.5
- new net 3.3V5: C46.1, C47.2, D12.C, J54.9, JP49.2, PWR5.2, R98.2, U11.5, U12.10, U12.15, U12.23, U12.29, U12.36, U12.5
- new net 5V3: BYP3.2, C30.1, D7.5, F4.2, J36.10, Q13.2, Q14.2, Q15.2, Q16.2, R64.2, R65.1, R66.1, R67.1, R68.1, U7.1, U7.3
- new net 5V4: BYP4.2, C39.1, D9.5, F5.2, J45.10, Q17.2, Q18.2, Q19.2, Q20.2, R82.2, R83.1, R84.1, R85.1, R86.1, U9.1, U9.3
- new net 5V5: BYP5.2, C48.1, D11.5, F6.2, J54.10, Q21.2, Q22.2, Q23.2, Q24.2, R100.2, R101.1, R102.1, R103.1, R104.1, U11.1, U11.3
- new net CC10: J40.B5, R74.2
- new net CC11: J49.A5, R93.2
- new net CC12: J49.B5, R92.2
- new net CC7: J31.A5, R57.2
- new net CC8: J31.B5, R56.2
- new net CC9: J40.A5, R75.2
- new net CFG4: J36.7, R61.2, U8.25
- new net CFG5: J45.7, R79.2, U10.25
- new net CFG6: J54.7, R97.2, U12.25
- new net D_N3: D7.6, R71.1
- new net D_N4: D9.6, R89.1
- new net D_N5: D11.6, R107.1
- new net D_P3: D7.4, R72.1
- new net D_P4: D9.4, R90.1
- new net D_P5: D11.4, R108.1
- new net GND3: C28.2, C29.1, C30.2, C31.1, C32.1, C33.2, C34.2, C35.2, C36.2, D7.2, J28.1, J29.1, J30.1, J31.GND, J31.GND2, J31.SHLD1, J31.SHLD2, J31.SHLD3, J31.SHLD4, J32.GND, J33.GND, J34.GND, J35.GND, J36.1, LED4.C, R56.1, R57.1, R58.2, R60.1, R61.1, R63.1, U7.2, U8.11, U8.EP
- new net GND4: C37.2, C38.1, C39.2, C40.1, C41.1, C42.2, C43.2, C44.2, C45.2, D9.2, J37.1, J38.1, J39.1, J40.GND, J40.GND2, J40.SHLD1, J40.SHLD2, J40.SHLD3, J40.SHLD4, J41.GND, J42.GND, J43.GND, J44.GND, J45.1, LED5.C, R74.1, R75.1, R76.2, R78.1, R79.1, R81.1, U10.11, U10.EP, U9.2
- new net GND5: C46.2, C47.1, C48.2, C49.1, C50.1, C51.2, C52.2, C53.2, C54.2, D11.2, J46.1, J47.1, J48.1, J49.GND, J49.GND2, J49.SHLD1, J49.SHLD2, J49.SHLD3, J49.SHLD4, J50.GND, J51.GND, J52.GND, J53.GND, J54.1, LED6.C, R92.1, R93.1, R94.2, R96.1, R97.1, R99.1, U11.2, U12.11, U12.EP
- new net N$100: J51.VBUS, Q22.3
- new net N$101: J52.VBUS, Q23.3
- new net N$102: J53.VBUS, Q24.3
- new net N$103: BYP5.1, F6.1, J49.VBUS1, J49.VBUS2
- new net N$104: JP49.1, R106.2
- new net N$105: JP49.3, R105.2
- new net N$106: R107.2, U12.30
- new net N$107: R108.2, U12.31
- new net N$108: D12.A, J46.2, J47.2, J48.2
- new net N$55: LED4.A, R55.1
- new net N$56: PWR3.1, R55.2
- new net N$57: C31.2, R59.2, U8.33, Y4.3
- new net N$58: C32.2, R59.1, U8.32, Y4.1
- new net N$59: R58.1, U8.35
- new net N$60: R60.2, U8.28
- new net N$61: C33.1, U8.34
- new net N$62: C34.1, U8.14
- new net N$63: J32.VBUS, Q13.3
- new net N$64: J33.VBUS, Q14.3
- new net N$65: J34.VBUS, Q15.3
- new net N$66: J35.VBUS, Q16.3
- new net N$67: BYP3.1, F4.1, J31.VBUS1, J31.VBUS2
- new net N$68: JP29.1, R70.2
- new net N$69: JP29.3, R69.2
- new net N$70: R71.2, U8.30
- new net N$71: R72.2, U8.31
- new net N$72: D8.A, J28.2, J29.2, J30.2
- new net N$73: LED5.A, R73.1
- new net N$74: PWR4.1, R73.2
- new net N$75: C40.2, R77.2, U10.33, Y5.3
- new net N$76: C41.2, R77.1, U10.32, Y5.1
- new net N$77: R76.1, U10.35
- new net N$78: R78.2, U10.28
- new net N$79: C42.1, U10.34
- new net N$80: C43.1, U10.14
- new net N$81: J41.VBUS, Q17.3
- new net N$82: J42.VBUS, Q18.3
- new net N$83: J43.VBUS, Q19.3
- new net N$84: J44.VBUS, Q20.3
- new net N$85: BYP4.1, F5.1, J40.VBUS1, J40.VBUS2
- new net N$86: JP39.1, R88.2
- new net N$87: JP39.3, R87.2
- new net N$88: R89.2, U10.30
- new net N$89: R90.2, U10.31
- new net N$90: D10.A, J37.2, J38.2, J39.2
- new net N$91: LED6.A, R91.1
- new net N$92: PWR5.1, R91.2
- new net N$93: C49.2, R95.2, U12.33, Y6.3
- new net N$94: C50.2, R95.1, U12.32, Y6.1
- new net N$95: R94.1, U12.35
- new net N$96: R96.2, U12.28
- new net N$97: C51.1, U12.34
- new net N$98: C52.1, U12.14
- new net N$99: J50.VBUS, Q21.3
- new net PORT1_N3: J32.D-, U8.1
- new net PORT1_N4: J41.D-, U10.1
- new net PORT1_N5: J50.D-, U12.1
- new net PORT1_P3: J32.D+, U8.2
- new net PORT1_P4: J41.D+, U10.2
- new net PORT1_P5: J50.D+, U12.2
- new net PORT2_N3: J33.D-, U8.3
- new net PORT2_N4: J42.D-, U10.3
- new net PORT2_N5: J51.D-, U12.3
- new net PORT2_P3: J33.D+, U8.4
- new net PORT2_P4: J42.D+, U10.4
- new net PORT2_P5: J51.D+, U12.4
- new net PORT3_N3: J34.D-, U8.6
- new net PORT3_N4: J43.D-, U10.6
- new net PORT3_N5: J52.D-, U12.6
- new net PORT3_P3: J34.D+, U8.7
- new net PORT3_P4: J43.D+, U10.7
- new net PORT3_P5: J52.D+, U12.7
- new net PORT4_N3: J35.D-, U8.8
- new net PORT4_N4: J44.D-, U10.8
- new net PORT4_N5: J53.D-, U12.8
- new net PORT4_P3: J35.D+, U8.9
- new net PORT4_P4: J44.D+, U10.9
- new net PORT4_P5: J53.D+, U12.9
- new net PRTPWR13: Q13.1, R65.2, U8.12
- new net PRTPWR14: Q14.1, R66.2, U8.16
- new net PRTPWR15: Q15.1, R67.2, U8.18
- new net PRTPWR16: Q16.1, R68.2, U8.20
- new net PRTPWR17: Q17.1, R83.2, U10.12
- new net PRTPWR18: Q18.1, R84.2, U10.16
- new net PRTPWR19: Q19.1, R85.2, U10.18
- new net PRTPWR20: Q20.1, R86.2, U10.20
- new net PRTPWR21: Q21.1, R101.2, U12.12
- new net PRTPWR22: Q22.1, R102.2, U12.16
- new net PRTPWR23: Q23.1, R103.2, U12.18
- new net PRTPWR24: Q24.1, R104.2, U12.20
- new net SCL/CFG3: J28.4, J29.4, J30.4, J36.8, R70.1, U8.24
- new net SCL/CFG4: J37.4, J38.4, J39.4, J45.8, R88.1, U10.24
- new net SCL/CFG5: J46.4, J47.4, J48.4, J54.8, R106.1, U12.24
- new net SDA3: J28.3, J29.3, J30.3, R69.1, U8.22
- new net SDA4: J37.3, J38.3, J39.3, R87.1, U10.22
- new net SDA5: J46.3, J47.3, J48.3, R105.1, U12.22
- new net UNP_D+3: D7.3, J31.A6, J31.B6
- new net UNP_D+4: D9.3, J40.A6, J40.B6
- new net UNP_D+5: D11.3, J49.A6, J49.B6
- new net UNP_D-3: D7.1, J31.A7, J31.B7
- new net UNP_D-4: D9.1, J40.A7, J40.B7
- new net UNP_D-5: D11.1, J49.A7, J49.B7
- new net VBUS_DET3: C36.1, R63.2, R64.1, U8.27
- new net VBUS_DET4: C45.1, R81.2, R82.1, U10.27
- new net VBUS_DET5: C54.1, R100.1, R99.2, U12.27
Routing:
- net SCL/CFG5: track 0.00 -> 143.6 mm, vias 0 -> 7
- net SCL/CFG4: track 0.00 -> 143.6 mm, vias 0 -> 7
- net SCL/CFG3: track 0.00 -> 143.6 mm, vias 0 -> 7
- net 5V5: track 0.00 -> 140.2 mm, vias 0 -> 12
- net 5V4: track 0.00 -> 140.2 mm, vias 0 -> 12
- net 5V3: track 0.00 -> 140.2 mm, vias 0 -> 12
- net 3.3V5: track 0.00 -> 139.8 mm, vias 0 -> 11
- net 3.3V3: track 0.00 -> 139.8 mm, vias 0 -> 11
- net 3.3V4: track 0.00 -> 139.8 mm, vias 0 -> 11
- net SDA5: track 0.00 -> 112.6 mm, vias 0 -> 5
- net SDA4: track 0.00 -> 112.6 mm, vias 0 -> 5
- net SDA3: track 0.00 -> 112.6 mm, vias 0 -> 5
- net N$108: track 0.00 -> 89.6 mm, vias 0 -> 2
- net N$90: track 0.00 -> 89.6 mm, vias 0 -> 2
- net N$72: track 0.00 -> 89.6 mm, vias 0 -> 2
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- added copper zone on layer 1, net GND3
- added copper zone on layer 16, net GND3
- added copper zone on layer 1, net GND4
- added copper zone on layer 16, net GND4
- added copper zone on layer 1, net GND5
- added copper zone on layer 16, net GND5
Other:
- board size 189.2 x 95 mm -> 189.2 x 176.8 mm
